File: hardware/dimmer/dimmer.kicad_sch (KiCad schematic)
At the start: 0 parts

Commit message: Capture dimmer + remote board schematics
Populate the previously-blank KiCad schematics for both boards per the
project spec, and add the Python generators that bootstrapped them.

Dimmer (mains, isolated): ESP32-WROOM-32, HLK-PM03 PSU, AC in/out screw
terminals, TLP281-4 zero-cross detect (R1/D1/R2 -> GPIO34), MOC3021 opto-TRIAC
gate drive (R3 <- GPIO25), BT138-600 TRIAC + gate resistor + RC snubber,
CP2102 USB-serial with USB-C and two-transistor auto-reset. Mains nets kept
separate from the 3V3/GND logic domain (isolation barrier).

Remote (battery): USB-C -> TP4056 charger -> LiPo -> ME6211 LDO -> 3V3 rail,
ESP32-WROOM-32, three tactile buttons on RTC GPIOs (39/34/35) each with a 100k
pull-up and 100nF debounce for low deep-sleep leakage, CP2102 USB-serial with
auto-reset.

Symbols use real KiCad stdlib parts where available and custom datasheet-
accurate symbols (HLK-PM03, TLP281-4, MOC3021, CP2102, ME6211, TP4056) where
not. Both schematics load in kicad-cli and the KiCad-computed netlist matches
the intended connectivity; the only unconnected pins are spare ESP32 GPIOs.

Files are KiCad-7 schematic format (20230121); KiCad 9/10 opens and upgrades.
Parts:
- added C1, C4: 10uF, Capacitor_SMD:C_1206_3216Metric, symbol Device:C
- added C2, C3, C7: 100nF, Capacitor_SMD:C_0805_2012Metric, symbol Device:C
- added C5: 100nF/X2, Capacitor_THT:C_Rect_L11.5mm_W5.0mm_P7.50mm_FKS3, symbol Device:C
- added C6: 1uF, Capacitor_SMD:C_0805_2012Metric, symbol Device:C
- added D1: 1N4007, Diode_THT:D_DO-41_SOD81_P10.16mm_Horizontal, symbol Diode:1N4007
- added J1: AC_IN_L_N, TerminalBlock_Phoenix:TerminalBlock_Phoenix_MKDS-1,5-2-5.08_1x02_P5.08mm_Horizontal, symbol Connector:Screw_Terminal_01x02
- added J2: AC_OUT_LOAD, TerminalBlock_Phoenix:TerminalBlock_Phoenix_MKDS-1,5-2-5.08_1x02_P5.08mm_Horizontal, symbol Connector:Screw_Terminal_01x02
- added J3: USB-C, Connector_USB:USB_C_Receptacle_HRO_TYPE-C-31-M-12, symbol Connector:USB_C_Receptacle_USB2.0_16P
- added PS1: HLK-PM03, Converter_ACDC:Converter_ACDC_HiLink_HLK-PMxx, symbol Power:HLK-PM03
- added Q1: BT138-600, Package_TO_SOT_THT:TO-220-3_Vertical, symbol Triac_Thyristor:BT138-600
- added Q2, Q3: MMBT3904, Package_TO_SOT_SMD:SOT-23, symbol Transistor_BJT:MMBT3904
- added R1: 10k, Resistor_THT:R_Axial_DIN0207_L6.3mm_D2.5mm_P10.16mm_Horizontal, symbol Device:R
- added R10, R9: 5.1k, Resistor_SMD:R_0805_2012Metric, symbol Device:R
- added R2, R6, R7, R8: 10k, Resistor_SMD:R_0805_2012Metric, symbol Device:R
- added R3: 330, Resistor_SMD:R_0805_2012Metric, symbol Device:R
- added R4: 470, Resistor_SMD:R_0805_2012Metric, symbol Device:R
- added R5: 47, Resistor_THT:R_Axial_DIN0207_L6.3mm_D2.5mm_P10.16mm_Horizontal, symbol Device:R
- added SW1: BOOT, Button_Switch_SMD:SW_SPST_PTS645, symbol Switch:SW_Push
- added SW2: EN, Button_Switch_SMD:SW_SPST_PTS645, symbol Switch:SW_Push
- added U1: ESP32-WROOM-32, RF_Module:ESP32-WROOM-32, symbol RF_Module:ESP32-WROOM-32
- added U2: TLP281-4, Package_SO:SOIC-16_3.9x9.9mm_P1.27mm, symbol Isolator:TLP281-4
- added U3: MOC3021, Package_DIP:DIP-6_W7.62mm, symbol Isolator:MOC3021
- added U4: CP2102, Package_DFN_QFN:QFN-28-1EP_5x5mm_P0.5mm, symbol Interface_USB:CP2102
Connections:
- new net +3V3: C1.1, C2.1, C4.1, PS1.4 (+Vo), R2.2, R6.1, R7.1, U1.2 (VDD)
- new net +5V: C6.1, J3.A4 (VBUS), J3.A9 (VBUS), J3.B4 (VBUS), J3.B9 (VBUS), U4.7 (REGIN), U4.8 (VBUS)
- new net AC_L_IN: J1.1 (Pin_1), PS1.1 (L~), Q1.2 (A2), R1.1, R5.1, U3.6 (MT)
- new net AC_L_OUT: C5.2, J2.1 (Pin_1), Q1.1 (A1)
- new net AC_N: D1.2 (A), J1.2 (Pin_2), J2.2 (Pin_2), PS1.2 (N~), U2.2 (K1)
- new net BOOT: Q3.3 (C), R7.2, SW1.1, U1.25 (IO0)
- new net CC1: J3.A5 (CC1), R9.1
- new net CC2: J3.B5 (CC2), R10.1
- new net CP_RST: R8.1, U4.9 (~{RST})
- new net DTR: Q2.1 (B), Q3.2 (E), U4.27 (DTR)
- new net EN: C3.1, Q2.3 (C), R6.2, SW2.1, U1.3 (EN)
- new net GATE_DRV: R3.1, U1.10 (IO25)
- new net GND: C1.2, C2.2, C3.2, C4.2, C6.2, C7.2, J3.A1 (GND), J3.A12 (GND), J3.B1 (GND), J3.B12 (GND), J3.S1 (SHIELD), PS1.3 (-Vo), R10.2, R9.2, SW1.2, SW2.2, U1.1 (GND), U1.15 (GND), U1.38 (GND), U1.39 (GND), U2.15 (E1), U3.2 (K), U4.3 (GND)
- new net MOC_LED_A: R3.2, U3.1 (A)
- new net MOC_MT: R4.1, U3.4 (MT)
- new net RTS: Q2.2 (E), Q3.1 (B), U4.24 (RTS)
- new net SNUB: C5.1, R5.2
- new net TRIAC_G: Q1.3 (G), R4.2
- new net U0RXD: U1.34 (RXD0/IO3), U4.26 (TXD)
- new net U0TXD: U1.35 (TXD0/IO1), U4.25 (RXD)
- new net USB_DM: J3.A7 (D-), J3.B7 (D-), U4.5 (D-)
- new net USB_DP: J3.A6 (D+), J3.B6 (D+), U4.4 (D+)
- new net V3V3_USB: C7.1, R8.2, U4.6 (VDD)
- new net ZC_DET: R2.1, U1.6 (IO34), U2.16 (C1)
- new net ZC_LED_A: D1.1 (K), R1.2, U2.1 (A1)
- no-connect marks 0 -> 40
Other:
- note added: "=== LOGIC 3V3 ==="
- note added: "=== MAINS 230V (ISOLATED) ==="
- note added: "ISOLATION BARRIER: routed slot under U2/U3 - no copper crosses (AC_ nets vs GND/3V3)"
- note added: "Opto-TRIAC gate drive <- GPIO25"
- note added: "USB-Serial + auto-reset"
- note added: "Zero-cross detect -> GPIO34"
