File: hardware/remote/remote.kicad_sch (KiCad schematic)
At the start: 0 parts

Commit message: Capture dimmer + remote board schematics
Populate the previously-blank KiCad schematics for both boards per the
project spec, and add the Python generators that bootstrapped them.

Dimmer (mains, isolated): ESP32-WROOM-32, HLK-PM03 PSU, AC in/out screw
terminals, TLP281-4 zero-cross detect (R1/D1/R2 -> GPIO34), MOC3021 opto-TRIAC
gate drive (R3 <- GPIO25), BT138-600 TRIAC + gate resistor + RC snubber,
CP2102 USB-serial with USB-C and two-transistor auto-reset. Mains nets kept
separate from the 3V3/GND logic domain (isolation barrier).

Remote (battery): USB-C -> TP4056 charger -> LiPo -> ME6211 LDO -> 3V3 rail,
ESP32-WROOM-32, three tactile buttons on RTC GPIOs (39/34/35) each with a 100k
pull-up and 100nF debounce for low deep-sleep leakage, CP2102 USB-serial with
auto-reset.

Symbols use real KiCad stdlib parts where available and custom datasheet-
accurate symbols (HLK-PM03, TLP281-4, MOC3021, CP2102, ME6211, TP4056) where
not. Both schematics load in kicad-cli and the KiCad-computed netlist matches
the intended connectivity; the only unconnected pins are spare ESP32 GPIOs.

Files are KiCad-7 schematic format (20230121); KiCad 9/10 opens and upgrades.
Parts:
- added BT1: LiPo_500mAh, Connector_JST:JST_PH_S2B-PH-SM4-TB_1x02-1MP_P2.00mm_Horizontal, symbol Connector_Generic:Conn_01x02
- added C10, C2, C3: 1uF, Capacitor_SMD:C_0805_2012Metric, symbol Device:C
- added C11, C5, C6, C7, C8, C9: 100nF, Capacitor_SMD:C_0805_2012Metric, symbol Device:C
- added C4: 10uF, Capacitor_SMD:C_1206_3216Metric, symbol Device:C
- added J1: USB-C, Connector_USB:USB_C_Receptacle_HRO_TYPE-C-31-M-12, symbol Connector:USB_C_Receptacle_USB2.0_16P
- added LED1: CHRG, LED_SMD:LED_0805_2012Metric, symbol Device:LED
- added LED2: FULL, LED_SMD:LED_0805_2012Metric, symbol Device:LED
- added Q1, Q2: MMBT3904, Package_TO_SOT_SMD:SOT-23, symbol Transistor_BJT:MMBT3904
- added R1: 1.2k, Resistor_SMD:R_0805_2012Metric, symbol Device:R
- added R10, R11: 5.1k, Resistor_SMD:R_0805_2012Metric, symbol Device:R
- added R2, R3: 1k, Resistor_SMD:R_0805_2012Metric, symbol Device:R
- added R4, R5, R6: 100k, Resistor_SMD:R_0805_2012Metric, symbol Device:R
- added R7, R8, R9: 10k, Resistor_SMD:R_0805_2012Metric, symbol Device:R
- added SW1: UP, Button_Switch_SMD:SW_SPST_PTS645, symbol Switch:SW_Push
- added SW2: DOWN, Button_Switch_SMD:SW_SPST_PTS645, symbol Switch:SW_Push
- added SW3: ON/OFF, Button_Switch_SMD:SW_SPST_PTS645, symbol Switch:SW_Push
- added U1: TP4056, Package_SO:SOIC-8_3.9x4.9mm_P1.27mm, symbol Battery_Management:TP4056
- added U2: ME6211C33M5G, Package_TO_SOT_SMD:SOT-23-5, symbol Regulator_Linear:ME6211C33
- added U3: ESP32-WROOM-32, RF_Module:ESP32-WROOM-32, symbol RF_Module:ESP32-WROOM-32
- added U4: CP2102, Package_DFN_QFN:QFN-28-1EP_5x5mm_P0.5mm, symbol Interface_USB:CP2102
Connections:
- new net +3V3: C3.1, C4.1, C5.1, R4.1, R5.1, R6.1, R7.1, R8.1, U2.5 (VOUT), U3.2 (VDD)
- new net +5V: C10.1, J1.A4 (VBUS), J1.A9 (VBUS), J1.B4 (VBUS), J1.B9 (VBUS), R2.1, R3.1, U1.4 (VCC), U1.8 (CE), U4.7 (REGIN), U4.8 (VBUS)
- new net BOOT: Q2.3 (C), R8.2, U3.25 (IO0)
- new net BTN_DOWN: C7.1, R5.2, SW2.1, U3.6 (IO34)
- new net BTN_ONOFF: C8.1, R6.2, SW3.1, U3.7 (IO35)
- new net BTN_UP: C6.1, R4.2, SW1.1, U3.5 (SENSOR_VN)
- new net CC1: J1.A5 (CC1), R10.1
- new net CC2: J1.B5 (CC2), R11.1
- new net CHRG_N: LED1.1 (K), U1.7 (~{CHRG})
- new net CP_RST: R9.1, U4.9 (~{RST})
- new net DTR: Q1.1 (B), Q2.2 (E), U4.27 (DTR)
- new net EN: C9.1, Q1.3 (C), R7.2, U3.3 (EN)
- new net GND: BT1.2 (Pin_2), C10.2, C11.2, C2.2, C3.2, C4.2, C5.2, C6.2, C7.2, C8.2, C9.2, J1.A1 (GND), J1.A12 (GND), J1.B1 (GND), J1.B12 (GND), J1.S1 (SHIELD), R1.2, R10.2, R11.2, SW1.2, SW2.2, SW3.2, U1.1 (TEMP), U1.3 (GND), U2.2 (GND), U3.1 (GND), U3.15 (GND), U3.38 (GND), U3.39 (GND), U4.3 (GND)
- new net LED_CHRG_A: LED1.2 (A), R2.2
- new net LED_STBY_A: LED2.2 (A), R3.2
- new net PROG: R1.1, U1.2 (PROG)
- new net RTS: Q1.2 (E), Q2.1 (B), U4.24 (RTS)
- new net STBY_N: LED2.1 (K), U1.6 (~{STDBY})
- new net U0RXD: U3.34 (RXD0/IO3), U4.26 (TXD)
- new net U0TXD: U3.35 (TXD0/IO1), U4.25 (RXD)
- new net USB_DM: J1.A7 (D-), J1.B7 (D-), U4.5 (D-)
- new net USB_DP: J1.A6 (D+), J1.B6 (D+), U4.4 (D+)
- new net V3V3_USB: C11.1, R9.2, U4.6 (VDD)
- new net VBAT: BT1.1 (Pin_1), C2.1, U1.5 (BAT), U2.1 (VIN), U2.3 (EN)
- no-connect marks 0 -> 27
Other:
- note added: "=== CHARGE + POWER ==="
- note added: "=== MCU (deep sleep, ext1 wake) ==="
- note added: "Buttons: 100k pull-up (low sleep leakage) + 100nF debounce"
- note added: "Target deep-sleep current ~5uA -> ~4-6 month battery life"
- note added: "USB-Serial + auto-reset"
